Commit message: racer找路失败

File: gazebo/lidar.xacro (robot description, xacro)
@@ -1,14 +1,13 @@
 <robot name="lidar" xmlns:xacro="http://wiki.ros.org/xacro">
     <xacro:property name="support_radius" value="0.01" />
-    <xacro:property name="support_length" value="0.3" />
+    <xacro:property name="support_length" value="0.15" />
     <xacro:property name="laser_radius" value="0.03" />
     <xacro:property name="laser_length" value="0.05" />
     <xacro:property name="support_off_x" value="0" />
     <xacro:property name="support_off_y" value="0" />
-    <xacro:property name="support_off_z" value="${ base_length/2 + laser_length/2 }" />
+    <xacro:property name="support_off_z" value="0.6" />
     <xacro:property name="lidar_off_x" value="0" />
     <xacro:property name="lidar_off_y" value="0" />
-    <!-- <xacro:property name="lidar_off_z" value="0.5" /> -->
-    <xacro:property name="lidar_off_z" value="${support_length/2 + laser_length/2}" />
+    <xacro:property name="lidar_off_z" value="${support_off_z/2 + laser_length/2}" />
     <link name="support">
         <visual>
