Commit message: gazebo success by 2D A*

File: gazebo/kinect.xacro (robot description, xacro)
@@ -13,6 +13,6 @@
                 </image>
                 <clip>
-                    <near>0.05</near>
-                    <far>8.0</far>
+                    <near>0.01</near>
+                    <far>10.0</far>
                 </clip>
             </camera>
@@ -33,5 +33,5 @@
                 <distortion_t1>0.0</distortion_t1>
                 <distortion_t2>0.0</distortion_t2>
-                <pointCloudCutoff>0.4</pointCloudCutoff>
+                <pointCloudCutoff>0.1</pointCloudCutoff>
             </plugin>
         </sensor>

File: gazebo/lidar.xacro (robot description, xacro)
@@ -6,5 +6,5 @@
     <xacro:property name="support_off_x" value="0" />
     <xacro:property name="support_off_y" value="0" />
-    <xacro:property name="support_off_z" value="0.6" />
+    <xacro:property name="support_off_z" value="0.4" />
     <xacro:property name="lidar_off_x" value="0" />
     <xacro:property name="lidar_off_y" value="0" />

File: gazebo/racer.xacro (robot description, xacro)
@@ -4,7 +4,7 @@
     <!-- <xacro:include filename="cam.xacro" /> -->
     <xacro:include filename="lidar.xacro" />
-    <xacro:include filename="/home/zqh/phoenixZ/racer_explore/gazebo/move.xacro"/>
-    <xacro:include filename="/home/zqh/phoenixZ/racer_explore/gazebo/laser.xacro"/>
-    <!-- <xacro:include filename="/home/zqh/phoenixZ/racer_explore/gazebo/camera.xacro"/> -->
-    <xacro:include filename="/home/zqh/phoenixZ/racer_explore/gazebo/kinect.xacro"/>
+    <xacro:include filename="/root/jky/racer_explore/gazebo/move.xacro"/>
+    <xacro:include filename="/root/jky/racer_explore/gazebo/laser.xacro"/>
+    <!-- <xacro:include filename="/root/jky/racer_explore/gazebo/camera.xacro"/> -->
+    <xacro:include filename="/root/jky/racer_explore/gazebo/kinect.xacro"/>
 </robot>

Commit message: 两车gazebo,2号车搜索失败容易撞车

File: gazebo/kinect.xacro (robot description, xacro)
@@ -33,5 +33,5 @@
                 <distortion_t1>0.0</distortion_t1>
                 <distortion_t2>0.0</distortion_t2>
-                <pointCloudCutoff>0.1</pointCloudCutoff>
+                <pointCloudCutoff>0.2</pointCloudCutoff>
             </plugin>
         </sensor>

File: gazebo/racer.xacro (robot description, xacro)
@@ -1,10 +1,387 @@
-<robot name="mycarwithlidarandcamera" xmlns:xacro="http://wiki.ros.org/xacro">
-    <xacro:include filename="interial.xacro" />
-    <xacro:include filename="car.xacro" />
-    <!-- <xacro:include filename="cam.xacro" /> -->
-    <xacro:include filename="lidar.xacro" />
-    <xacro:include filename="/root/jky/racer_explore/gazebo/move.xacro"/>
-    <xacro:include filename="/root/jky/racer_explore/gazebo/laser.xacro"/>
-    <!-- <xacro:include filename="/root/jky/racer_explore/gazebo/camera.xacro"/> -->
-    <xacro:include filename="/root/jky/racer_explore/gazebo/kinect.xacro"/>
+<robot xmlns:xacro="http://wiki.ros.org/xacro" name="$(arg prefix)mycarwithlidarandcamera">
+    <!-- 定义参数 -->
+    <xacro:arg name="prefix" default="" />
+    <xacro:arg name="namespace" default="" />
+    <!-- 属性定义 -->
+    <xacro:property name="footprint_radius" value="0.003"/>
+    <xacro:property name="base_radius" value="0.3"/>
+    <xacro:property name="base_length" value="0.24"/>
+    <xacro:property name="lidi" value="0.045"/>
+    <xacro:property name="base_joint_z" value="${base_length/2 + lidi}"/>
+    <xacro:property name="wheel_radius" value="0.0975"/>
+    <xacro:property name="wheel_length" value="0.045"/>
+    <xacro:property name="PI" value="3.1415927"/>
+    <xacro:property name="wheel_joint_Z" value="${-base_length/2 - lidi + wheel_radius}"/>
+    <xacro:property name="small_radius" value="0.0225"/>
+    <xacro:property name="small_jointz" value="${-base_length/2 - lidi + small_radius}"/>
+    <xacro:property name="cam_x" value="0.02" />
+    <xacro:property name="cam_y" value="0.05" />
+    <xacro:property name="cam_z" value="0.05" />
+    <xacro:property name="cam_off_x" value="0.24" />
+    <xacro:property name="cam_off_y" value="0" />
+    <xacro:property name="cam_off_z" value="0.245" />
+    <xacro:property name="support_radius" value="0.01" />
+    <xacro:property name="support_length" value="0.3" />
+    <xacro:property name="laser_radius" value="0.03" />
+    <xacro:property name="laser_length" value="0.05" />
+    <xacro:property name="support_off_x" value="0" />
+    <xacro:property name="support_off_y" value="0" />
+    <xacro:property name="support_off_z" value="0.4" />
+    <xacro:property name="lidar_off_x" value="0" />
+    <xacro:property name="lidar_off_y" value="0" />
+    <xacro:property name="lidar_off_z" value="${support_length/2 + laser_length/2}" />
+    <!-- 惯性矩阵宏定义 -->
+    <xacro:macro name="sphere_inertial_matrix" params="m r">
+        <inertial>
+            <mass value="${m}" />
+            <inertia ixx="${2*m*r*r/5}" ixy="0" ixz="0"
+                     iyy="${2*m*r*r/5}" iyz="0"
+                     izz="${2*m*r*r/5}" />
+        </inertial>
+    </xacro:macro>
+    <xacro:macro name="cylinder_inertial_matrix" params="m r h">
+        <inertial>
+            <mass value="${m}" />
+            <inertia ixx="${m*(3*r*r+h*h)/12}" ixy="0" ixz="0"
+                     iyy="${m*(3*r*r+h*h)/12}" iyz="0"
+                     izz="${m*r*r/2}" />
+        </inertial>
+    </xacro:macro>
+    <xacro:macro name="Box_inertial_matrix" params="m l w h">
+        <inertial>
+            <mass value="${m}" />
+            <inertia ixx="${m*(h*h + l*l)/12}" ixy="0" ixz="0"
+                     iyy="${m*(w*w + l*l)/12}" iyz="0"
+                     izz="${m*(w*w + h*h)/12}" />
+        </inertial>
+    </xacro:macro>
+    <!-- 车轮宏定义 -->
+    <xacro:macro name="wheel_func" params="wheel_name flag">
+        <link name="$(arg prefix)${wheel_name}_wheel">
+            <visual>
+                <geometry>
+                    <cylinder radius="${wheel_radius}" length="${wheel_length}" />
+                </geometry>
+                <origin xyz="0 0 0" rpy="${PI/2} 0 0" />
+                <material name="wheel_color">
+                    <color rgba="0 0 1.0 0.5 0.3" />
+                </material>
+            </visual>
+            <collision>
+                <geometry>
+                    <cylinder radius="${wheel_radius}" length="${wheel_length}" />
+                </geometry>
+                <origin xyz="0.0 0.0 0.0" rpy="${PI / 2} 0.0 0.0" />
+            </collision>
+            <xacro:cylinder_inertial_matrix m="9" r="${wheel_radius}" h="${wheel_length}" />
+        </link>
+        <joint name="$(arg prefix)base_link2_${wheel_name}" type="continuous">
+            <parent link="$(arg prefix)base_link" />
+            <child link="$(arg prefix)${wheel_name}_wheel"/>
+            <origin xyz="0 ${0.3 * flag} ${wheel_joint_Z}" />
+            <axis xyz="0 1 0" />
+        </joint>
+        <gazebo reference="$(arg prefix)${wheel_name}_wheel">
+            <material>Gazebo/Red</material>
+        </gazebo>
+    </xacro:macro>
+    <xacro:macro name="small_wheel_func" params="small_wheel_name flag">
+        <link name="$(arg prefix)${small_wheel_name}_wheel">
+            <visual>
+                <geometry>
+                    <sphere radius="${small_radius}" />
+                </geometry>
+                <origin xyz="0 0 0" rpy="0 0 0" />
+                <material name="black">
+                    <color rgba="0.0 0.0 0.0 0.6" />
+                </material>
+            </visual>
+            <collision>
+                <geometry>
+                    <sphere radius="${small_radius}" />
+                </geometry>
+                <origin xyz="0 0 0" rpy="0 0 0" />
+            </collision>
+            <xacro:sphere_inertial_matrix m="0.72" r="${small_radius}" />
+        </link>
+        <joint name="$(arg prefix)${small_wheel_name}2base_link" type="continuous">
+            <parent link="$(arg prefix)base_link" />
+            <child link="$(arg prefix)${small_wheel_name}_wheel" />
+            <origin xyz="${0.2775 * flag} 0 ${small_jointz}" />
+            <axis xyz="1 1 1" />
+        </joint>
+        <gazebo reference="$(arg prefix)${small_wheel_name}_wheel">
+            <material>Gazebo/Red</material>
+        </gazebo>
+    </xacro:macro>
+    <!-- 驱动宏定义 -->
+    <xacro:macro name="joint_trans" params="joint_name">
+        <transmission name="$(arg prefix)${joint_name}_trans">
+            <type>transmission_interface/SimpleTransmission</type>
+            <joint name="$(arg prefix)${joint_name}">
+                <hardwareInterface>hardware_interface/VelocityJointInterface</hardwareInterface>
+            </joint>
+            <actuator name="$(arg prefix)${joint_name}_motor">
+                <hardwareInterface>hardware_interface/VelocityJointInterface</hardwareInterface>
+                <mechanicalReduction>1</mechanicalReduction>
+            </actuator>
+        </transmission>
+    </xacro:macro>
+    <!-- 链接和关节定义 -->
+    <!-- base_footprint -->
+    <link name="$(arg prefix)base_footprint">
+        <visual>
+            <geometry>
+                <sphere radius="${footprint_radius}" />
+            </geometry>
+        </visual>
+    </link>
+    <!-- base_link -->
+    <link name="$(arg prefix)base_link">
+        <visual>
+            <geometry>
+                <cylinder radius="${base_radius}" length="${base_length}" />
+            </geometry>
+            <origin xyz="0 0 0" rpy="0 0 0" />
+            <material name="blue">
+                <color rgba="0 0 1.0 0.5" />
+            </material>
+        </visual>
+        <collision>
+            <geometry>
+                <cylinder radius="${base_radius}" length="${base_length}" />
+            </geometry>
+            <origin xyz="0 0 0" rpy="0 0 0" />
+        </collision>
+        <xacro:cylinder_inertial_matrix m="18" r="${base_radius}" h="${base_length}" />
+    </link>
+    <gazebo reference="$(arg prefix)base_link">
+        <material>Gazebo/Yellow</material>
+    </gazebo>
+    <joint name="$(arg prefix)base_link2base_footprint" type="fixed">
+        <parent link="$(arg prefix)base_footprint" />
+        <child link="$(arg prefix)base_link"/>
+        <origin xyz="0 0 ${base_joint_z}" />
+    </joint>
+    <!-- 车轮实例化 -->
+    <xacro:wheel_func wheel_name="left" flag="1" />
+    <xacro:wheel_func wheel_name="right" flag="-1" />
+    <xacro:small_wheel_func small_wheel_name="front" flag="1" />
+    <xacro:small_wheel_func small_wheel_name="back" flag="-1" />
+    <!-- camera -->
+    <!-- <link name="$(arg prefix)camera">
+        <visual>
+            <geometry>
+                <box size="${cam_x} ${cam_y} ${cam_z}" />
+            </geometry>
+            <origin xyz="0.0 0.0 0.0" rpy="0.0 0.0 0.0" />
+            <material name="black" />
+        </visual>
+        <collision>
+            <geometry>
+                <box size="${cam_x} ${cam_y} ${cam_z}" />
+            </geometry>
+            <origin xyz="0.0 0.0 0.0" rpy="0.0 0.0 0.0" />
+        </collision>
+        <xacro:Box_inertial_matrix m="0.01" l="${cam_x}" w="${cam_y}" h="${cam_z}" />
+    </link>
+    <joint name="$(arg prefix)camera2base_link" type="fixed">
+        <parent link="$(arg prefix)base_link" />
+        <child link="$(arg prefix)camera" />
+        <origin xyz="${cam_off_x} ${cam_off_y} ${cam_off_z}" />
+    </joint>
+    <gazebo reference="$(arg prefix)camera">
+        <material>Gazebo/Blue</material>
+    </gazebo> -->
+    <!-- support 和 laser -->
+    <link name="$(arg prefix)support">
+        <visual>
+            <geometry>
+                <cylinder radius="${support_radius}" length="${support_length}" />
+            </geometry>
+            <origin xyz="0.0 0.0 0.0" rpy="0.0 0.0 0.0" />
+            <material name="red">
+                <color rgba="0.8 0.2 0.0 0.8" />
+            </material>
+        </visual>
+        <collision>
+            <geometry>
+                <cylinder radius="${support_radius}" length="${support_length}" />
+            </geometry>
+            <origin xyz="0.0 0.0 0.0" rpy="0.0 0.0 0.0" />
+        </collision>
+        <xacro:cylinder_inertial_matrix m="0.1" r="${support_radius}" h="${support_length}" />
+    </link>
+    <gazebo reference="$(arg prefix)support">
+        <material>Gazebo/Grey</material>
+    </gazebo>
+    <joint name="$(arg prefix)support2base_link" type="fixed">
+        <parent link="$(arg prefix)base_link" />
+        <child link="$(arg prefix)support" />
+        <origin xyz="${support_off_x} ${support_off_y} ${support_off_z}" />
+    </joint>
+    <!-- 添加 support_depth 链接 -->
+    <link name="$(arg prefix)support_depth" />
+    <joint name="$(arg prefix)support2support_depth" type="fixed">
+        <parent link="$(arg prefix)support" />
+        <child link="$(arg prefix)support_depth" />
+        <origin xyz="0 0 0" rpy="${-PI/2} 0 ${-PI/2}" />
+    </joint>
+    <link name="$(arg prefix)laser">
+        <visual>
+            <geometry>
+                <cylinder radius="${laser_radius}" length="${laser_length}" />
+            </geometry>
+            <origin xyz="0.0 0.0 0.0" rpy="0.0 0.0 0.0" />
+            <material name="black" />
+        </visual>
+        <collision>
+            <geometry>
+                <cylinder radius="${laser_radius}" length="${laser_length}" />
+            </geometry>
+            <origin xyz="0.0 0.0 0.0" rpy="0.0 0.0 0.0" />
+        </collision>
+        <xacro:cylinder_inertial_matrix m="0.15" r="${laser_radius}" h="${laser_length}" />
+    </link>
+    <joint name="$(arg prefix)laser2support" type="fixed">
+        <parent link="$(arg prefix)support" />
+        <child link="$(arg prefix)laser" />
+        <origin xyz="${lidar_off_x} ${lidar_off_y} ${lidar_off_z}" />
+    </joint>
+    <gazebo reference="$(arg prefix)laser">
+        <material>Gazebo/Black</material>
+    </gazebo>
+    <!-- Gazebo 插件和传感器 -->
+    <!-- 驱动插件 -->
+    <xacro:joint_trans joint_name="base_link2_left" />
+    <xacro:joint_trans joint_name="base_link2_right" />
+    <gazebo>
+        <plugin name="$(arg prefix)differential_drive_controller" filename="libgazebo_ros_diff_drive.so">
+            <rosDebugLevel>Debug</rosDebugLevel>
+            <publishWheelTF>true</publishWheelTF>
+            <robotNamespace>$(arg namespace)</robotNamespace>
+            <publishTf>1</publishTf>
+            <publishWheelJointState>true</publishWheelJointState>
+            <alwaysOn>true</alwaysOn>
+            <updateRate>100.0</updateRate>
+            <legacyMode>true</legacyMode>
+            <leftJoint>$(arg prefix)base_link2_left</leftJoint>
+            <rightJoint>$(arg prefix)base_link2_right</rightJoint>
+            <wheelSeparation>${base_radius * 2}</wheelSeparation>
+            <wheelDiameter>${wheel_radius * 2}</wheelDiameter>
+            <broadcastTF>1</broadcastTF>
+            <wheelTorque>30</wheelTorque>
+            <wheelAcceleration>1.8</wheelAcceleration>
+            <commandTopic>$(arg namespace)/cmd_vel</commandTopic>
+            <odometryFrame>$(arg prefix)odom</odometryFrame>
+            <odometryTopic>$(arg namespace)/odom</odometryTopic>
+            <robotBaseFrame>$(arg prefix)base_footprint</robotBaseFrame>
+        </plugin>
+    </gazebo>
+    <!-- 摄像头传感器 -->
+    <!-- <gazebo reference="$(arg prefix)camera">
+        <sensor type="camera" name="$(arg prefix)camera_node">
+            <update_rate>30.0</update_rate>
+            <camera name="head">
+                <horizontal_fov>1.3962634</horizontal_fov>
+                <image>
+                    <width>1280</width>
+                    <height>720</height>
+                    <format>R8G8B8</format>
+                </image>
+                <clip>
+                    <near>0.02</near>
+                    <far>300</far>
+                </clip>
+                <noise>
+                    <type>gaussian</type>
+                    <mean>0.0</mean>
+                    <stddev>0.007</stddev>
+                </noise>
+            </camera>
+            <plugin name="$(arg prefix)gazebo_camera" filename="libgazebo_ros_camera.so">
+                <alwaysOn>true</alwaysOn>
+                <updateRate>0.0</updateRate>
+                <cameraName>$(arg namespace)/camera</cameraName>
+                <imageTopicName>$(arg namespace)/image_raw</imageTopicName>
+                <cameraInfoTopicName>$(arg namespace)/camera_info</cameraInfoTopicName>
+                <frameName>$(arg prefix)camera</frameName>
+                <hackBaseline>0.07</hackBaseline>
+                <distortionK1>0.0</distortionK1>
+                <distortionK2>0.0</distortionK2>
+                <distortionK3>0.0</distortionK3>
+                <distortionT1>0.0</distortionT1>
+                <distortionT2>0.0</distortionT2>
+            </plugin>
+        </sensor>
+    </gazebo> -->
+    <!-- 激光雷达传感器 -->
+    <gazebo reference="$(arg prefix)laser">
+        <sensor type="ray" name="$(arg prefix)rplidar">
+            <pose>0 0 0 0 0 0</pose>
+            <visualize>false</visualize>
+            <update_rate>5.5</update_rate>
+            <ray>
+                <scan>
+                    <horizontal>
+                        <samples>360</samples>
+                        <resolution>1</resolution>
+                        <min_angle>-3</min_angle>
+                        <max_angle>3</max_angle>
+                    </horizontal>
+                </scan>
+                <range>
+                    <min>0.10</min>
+                    <max>30.0</max>
+                    <resolution>0.01</resolution>
+                </range>
+                <noise>
+                    <type>gaussian</type>
+                    <mean>0.0</mean>
+                    <stddev>0.01</stddev>
+                </noise>
+            </ray>
+            <plugin name="$(arg prefix)gazebo_rplidar" filename="libgazebo_ros_laser.so">
+                <topicName>$(arg namespace)/scan</topicName>
+                <frameName>$(arg prefix)laser</frameName>
+            </plugin>
+        </sensor>
+    </gazebo>
+    <!-- Kinect 传感器 -->
+    <gazebo reference="$(arg prefix)support">
+        <sensor type="depth" name="$(arg prefix)kinect_camera">
+            <always_on>true</always_on>
+            <update_rate>20.0</update_rate>
+            <camera>
+                <horizontal_fov>${60.0*PI/180.0}</horizontal_fov>
+                <image>
+                    <format>R8G8B8</format>
+                    <width>640</width>
+                    <height>480</height>
+                </image>
+                <clip>
+                    <near>0.05</near>
+                    <far>10.0</far>
+                </clip>
+            </camera>
+            <plugin name="$(arg prefix)kinect_camera_controller" filename="libgazebo_ros_openni_kinect.so">
+                <cameraName>$(arg namespace)/camera</cameraName>
+                <alwaysOn>true</alwaysOn>
+                <updateRate>10</updateRate>
+                <imageTopicName>$(arg namespace)/rgb/image_raw</imageTopicName>
+                <depthImageTopicName>$(arg namespace)/depth/image_raw</depthImageTopicName>
+                <pointCloudTopicName>$(arg namespace)/depth/points</pointCloudTopicName>
+                <cameraInfoTopicName>$(arg namespace)/rgb/camera_info</cameraInfoTopicName>
+                <depthImageCameraInfoTopicName>$(arg namespace)/depth/camera_info</depthImageCameraInfoTopicName>
+                <frameName>$(arg prefix)support_depth</frameName>
+                <baseline>0.1</baseline>
+                <distortion_k1>0.0</distortion_k1>
+                <distortion_k2>0.0</distortion_k2>
+                <distortion_k3>0.0</distortion_k3>
+                <distortion_t1>0.0</distortion_t1>
+                <distortion_t2>0.0</distortion_t2>
+                <pointCloudCutoff>0.2</pointCloudCutoff>
+            </plugin>
+        </sensor>
+    </gazebo>
 </robot>
